File: hw/LED matrix/LED matrix.kicad_sch (KiCad schematic)
At the start: 62 parts, among them Q2 BS170, Q3 BS170, Q4 BS170, Q5 BS170, Q6 BS170, U1 STM32F103C6Tx, U2 74HC595, U3 74HC138

Commit message: Kapcsrajz finomítása és bővebb dokumentáció
Parts:
- added R15: 100k, symbol Device:R
Connections:
- net +3.3V: now also U3.16 (VCC), R15.1
- net GND: now also U3.4 (~{E0}), U3.5 (~{E1}), U3.8 (GND)
- net at R14.1: now also U3.11 (~{Y4})
- net at R7.1: now also U2.2 (QC)
- net at U3.12 (~{Y3}): now also R13.1
- net at U3.13 (~{Y2}): now also R12.1
- net at U3.14 (~{Y1}): now also R11.1
- net at U3.15 (~{Y0}): now also R10.1
- net at U3.6 (E2): now also R15.2
- net at U2.1 (QB): now also R6.1
- net at U2.15 (QA): now also R5.1
- net at U2.3 (QD): now also R8.1
- net at U2.4 (QE): now also R1.1
- net at U2.5 (QF): now also R3.1
- net at U2.6 (QG): now also R2.1
- net at U2.7 (QH): now also R4.1
- no-connect marks 36 -> 39
Other:
- note added: "Egy 5x8-as LED mátrix, amelyet STM32 fog vezérelni. Működése a standard LED mátrix működés. Folyamatosan váltogatjuk az oszlopokat olyan sebességgel, amellyel már egy képnek tűnik amit a mátrix mutat"
- note added: "Ez egy demultiplexer, amely a megfelelő oszlopot választja ki"
- note added: "Ez egy shift regiszter, amely egy oszlopon belül a megfelelő sorokat választja ki"
- note added: "Fontos megjegyzések: https://youtu.be/uQMUPhyoXoE https://youtu.be/Degt4HUzWXY"
- note added: "LED mátrix"
- note added: "MCU: Egy standard black pillel fogom megvalósítani"
- note added: "Áramnyelők, amelyeket a demultiplexer vezérel, egy kiválasztott oszlopban egy ilyen tranzisztor zárja az áramkört"
- moved on the sheet: D1, D10, D11, D12, D13, D14, D15, D16, D17, D18, D19, D2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

Commit message: A 74HC595-ös demultiplexer mégsem alkalmas az oszlop kiválasztására, mert invertálva vannak a kimenetei, ezt úgy oldottam meg, hogy azt is egy shift regiszter fogja helyettesíteni, de mivel az MCU-nak csak egy SPI channelje van, ezért ugyanazt a channel-t fogják használni, az RCLK lesz a slave kiválasztó jel
Parts:
- removed U3: 74HC138, symbol 74xx:74HC138
- added U3: 74HC595, symbol 74xx:74HC595
Connections:
- net +3.3V: now also U3.16 (VCC)
- net GND: now also U3.8 (GND); no longer U2.13 (~{OE})
- net SCK: now also U3.11 (SRCLK)
- net SData: now also U3.14 (SER)
- net at R14.1: now also U3.4 (QE)
- net at R13.1: now also U3.3 (QD)
- net at R12.1: now also U3.2 (QC)
- net at R11.1: now also U3.1 (QB)
- net at R10.1: now also U3.15 (QA)
- net at R15.2: now also U3.10 (~{SRCLR})
- net RCLK2: now reaches U1.14 (PA4)
- net RCLK2: now also U3.12 (RCLK)
- net RCLK1: now reaches U1.16 (PA6)
- net RCLK1: now also U2.12 (RCLK)
- net OEN: now reaches U1.18 (PB0)
- net OEN: now also U2.13 (~{OE}), U3.13 (~{OE})
- net PWM: no longer names the net of U1.32 (PA11)
- net RCLK: no longer names the net of U1.31 (PA10)
- net RCLK: no longer U2.12 (RCLK)
Other:
- note added: "Ez egy shift regiszter, amely a megfelelő oszlopot választja ki"
- note added: "Áramnyelők, amelyeket a shift regiszter vezérel, egy kiválasztott oszlopban egy ilyen tranzisztor zárja az áramkört"
- note removed: "Ez egy demultiplexer, amely a megfelelő oszlopot választja ki"
- note removed: "Áramnyelők, amelyeket a demultiplexer vezérel, egy kiválasztott oszlopban egy ilyen tranzisztor zárja az áramkört"
